File: hardware/v0a/v0a.brd (EAGLE design)
At the start: 100 x 100 mm, 263 parts, among them J1 2EDG-2P, J10 SH-5, J11 2EDG-2P, J12 SH-3, J13 SH-2, J14 F20F-10DP-1V, J15 SH-3, J16 SH-6, J2 2EDG-2P, J3 2EDG-2P, J4 2EDG-2P, J5 SH-5, J6 SH-5, J7 SH-5, J8 SH-5, J9 SH-2, Q1 IRF7580, Q2 IRF7580, Q3 IRF7580, Q4 IRF7580, Q5 IRF7580, Q6 IRF7580, Q7 IRF7580, Q8 IRF7580, Q9 IRF7580, U1 TMC4671, U10 AD8418, U11 AD8418, U12 DSC1101, U13 74LVC3G17, U14 74LVC3G17, U15 74LVC3G17, U16 74LVC3G17, U17 SI8261, U18 SRV05-4, U19 SRV05-4, U2 MIC39101, U20 SRV05-4, U21 SRV05-4, U3 MIC39101, U4 SI82397, U5 SI82397, U6 SI82397, U7 SI82397, U8 MIC4682, U9 CP2130

Commit message: pcb work
Parts:
- removed J4: 2EDG-2P, Connectors > Other:2EDG-2P
- added C16, C17, C32, C33, C46, C53: 100n, Passive Components > Capacitors > Multilayer Ceramic Capacitors MLCC:0603_WAVE
- added P1, P2, P3, P4: POWPAD, Connectors > Other:TH-HP
- added R96, R97, R98, R99: (no value), Passive Components > Resistors > Chip Resistors:0603_WAVE
- D1, D2, D3, D4: value SK54L -> DSK24; device Semiconductors > Discrete Semiconductors > Diodes & Rectifiers > Schottky Diodes & Rectifiers:DO214AA -> Semiconductors > Discrete Semiconductors > Diodes & Rectifiers > Schottky Diodes & Rectifiers:SOD-123
- J3: value 2EDG-2P -> 4P-6.35P; device Connectors > Other:2EDG-2P -> Connectors > Other:4P-6.35P
- U10, U11: value AD8418 -> AD8418A; device Semiconductors > Integrated Circuits - ICs > Amplifier ICs > Current Sense Amplifiers:SOIC8 -> Semiconductors > Integrated Circuits - ICs > Amplifier ICs > Current Sense Amplifiers:MSOP-8
- moved R31 194.5 mm to (92.1, 43.8), turned to 270 degrees
- moved R30 167.2 mm to (67.9, 43.8), turned to 270 degrees
- moved C38 144.0 mm to (92.1, 39.4), turned to 90 degrees
- moved R29 140.0 mm to (43.8, 43.8), turned to 270 degrees
- moved C37 117.6 mm to (67.9, 39.4), turned to 90 degrees
- moved R28 113.3 mm to (19.7, 43.8), turned to 270 degrees
- moved C70 94.8 mm to (43.2, 66.0), turned to 180 degrees
- moved C35 93.0 mm to (43.8, 39.4), turned to 90 degrees
- moved C69 88.2 mm to (43.2, 71.8)
- moved J3 77.3 mm to (52.1, 2.54)
- moved C34 71.8 mm to (19.7, 39.4), turned to 90 degrees
- moved R37 71.6 mm to (43.2, 67.9), turned to 180 degrees
- moved R36 67.5 mm to (43.2, 69.8)
- moved J14 20.7 mm to (56.5, 74.3)
- moved U1 8.41 mm to (50.0, 65.0), turned to 270 degrees
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Connections:
- new net N$10: R9.SENSE-, R96.P$1
- new net N$14: C16.P$1, C17.P$2, R96.P$2, U10.1
- new net N$18: C16.P$2, C32.P$1, R97.P$2, U10.8
- new net N$6: R9.SENSE+, R97.P$1
- net GND: now also C17.P$1, C32.P$2, C46.P$1, C53.P$2
- net N$28: now also J3.2, P2.H1, P2.H10, P2.H11, P2.H12, P2.H2, P2.H3, P2.H4, P2.H5, P2.H6, P2.H7, P2.H8, P2.H9, P2.PAD; no longer J3.P$2
- net N$29: now also J3.1, P1.H1, P1.H10, P1.H11, P1.H12, P1.H2, P1.H3, P1.H4, P1.H5, P1.H6, P1.H7, P1.H8, P1.H9, P1.PAD; no longer J3.P$1
- net N$55: now also R98.P$1; no longer U11.1
- net N$56: now also R99.P$1; no longer U11.8
- net N$57: now also C33.P$2, C53.P$1, R99.P$2, U11.8; no longer R9.SENSE-, U10.1
- net N$58: now also C33.P$1, C46.P$2, R98.P$2, U11.1; no longer R9.SENSE+, U10.8
- net WY1: now also J3.3, P3.H1, P3.H10, P3.H11, P3.H12, P3.H2, P3.H3, P3.H4, P3.H5, P3.H6, P3.H7, P3.H8, P3.H9, P3.PAD; no longer J4.P$1
- net Y2: now also J3.4, P4.H1, P4.H10, P4.H11, P4.H12, P4.H2, P4.H3, P4.H4, P4.H5, P4.H6, P4.H7, P4.H8, P4.H9, P4.PAD; no longer J4.P$2
Routing:
- net N$55: track 39.4 -> 0.00 mm
- net N$57: track 39.2 -> 0.00 mm
- net N$56: track 36.2 -> 0.00 mm
- net N$58: track 36.2 -> 0.00 mm
- net N$10: track 0.00 -> 35.4 mm, vias 1 -> 0
- net N$6: track 0.00 -> 35.3 mm, vias 1 -> 0
- net VX2: track 0.00 -> 18.2 mm
- net WY1: track 0.00 -> 18.2 mm
- net Y2: track 0.00 -> 18.0 mm
- net UX1: track 9.59 -> 18.2 mm
- net N$27: track 0.00 -> 6.04 mm
- net N$26: track 0.00 -> 5.98 mm
- net N$25: track 0.00 -> 5.98 mm
- net N$24: track 0.00 -> 5.98 mm
- net N$19: track 0.00 -> 4.72 mm
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- added copper zone on layer 1, net N$28
- added copper zone on layer 1, net N$29
- added copper zone on layer 1, net VX2
- added copper zone on layer 1, net WY1
- added copper zone on layer 1, net Y2
- removed copper zone on layer 1, net DCBUS1
- removed copper zone on layer 1, net GND1
- removed copper zone on layer 1, net GND2
- removed copper zone on layer 1, net GND3
- removed copper zone on layer 1, net UX2
- removed copper zone on layer 1, net UX3
- removed copper zone on layer 1, net UX4

Commit message: pcb work
Parts:
- removed C73, C74: 100n, Passive Components > Capacitors > Multilayer Ceramic Capacitors MLCC:0603_WAVE
- removed C75: 4u7, Passive Components > Capacitors > Multilayer Ceramic Capacitors MLCC:0603_WAVE
- removed D7: (no value), Opto-electronics > LED Emitters:CHIPLED_0603
- removed J11: 2EDG-2P, Connectors > Other:2EDG-2P
- removed R14: 10k, Passive Components > Resistors > Chip Resistors:0603_WAVE
- removed R44: (no value), Passive Components > Resistors > Chip Resistors:0603_WAVE
- added J4: 2P-6.35P, Connectors > Other:2P-6.35P
- added JP3, JP4, JP5, JP7: JUMPER-SMT_2_NC_PASTE_SILK, Utility > Board:SMT-JUMPER_2_NC_PASTE_SILK
- added JP6: JUMPER-SMT_2_NO_SILK, Utility > Board:SMT-JUMPER_2_NO_SILK
- added P5, P6, P7, P8: POWPAD, Connectors > Other:TH-HP
- added U$12, U$15, U$16: MOUNTINGHOLE3.0, Utility > Board:MOUNTINGHOLE_3.0_PLATED
- J1, J2: value 2EDG-2P -> 2P-6.35P; device Connectors > Other:2EDG-2P -> Connectors > Other:2P-6.35P
- JP1: value JUMPER-SMT_3_1-NC_PASTE_SILK -> JUMPER-SMT_2_NC_PASTE_SILK; device Utility > Board:SMT-JUMPER_3_1-NC_PASTE_SILK -> Utility > Board:SMT-JUMPER_2_NC_PASTE_SILK
- JP2: value JUMPER-SMT_3_1-NC_PASTE_SILK -> JUMPER-SMT_2_NO_SILK; device Utility > Board:SMT-JUMPER_3_1-NC_PASTE_SILK -> Utility > Board:SMT-JUMPER_2_NO_SILK
- U$13: value CP2102N -> MOUNTINGHOLE3.0; device Semiconductors > Integrated Circuits - ICs > Interface ICs > USB Interface IC:QFN24 -> Utility > Board:MOUNTINGHOLE_3.0_PLATED
- U9: value CP2130 -> CP2130/2102N
- moved R94 223.2 mm to (116.2, 85.7)
- moved R93 220.0 mm to (110.5, 78.1)
- moved R95 207.0 mm to (111.1, 85.7)
- moved J8 189.6 mm to (-141.0, 160.0)
- moved U16 180.4 mm to (-127.6, 156.2)
- moved C26 177.9 mm to (72.4, 95.2), turned to 90 degrees
- moved R24 176.7 mm to (102.2, 52.7), turned to 270 degrees
- moved R23 174.9 mm to (104.1, 52.7), turned to 270 degrees
- moved J6 165.9 mm to (-96.5, 149.9)
- moved U14 159.8 mm to (-87.0, 171.4)
- moved R33 158.1 mm to (50.8, 66.0)
- moved R27 154.6 mm to (69.2, 57.8), turned to 180 degrees
- moved R32 154.1 mm to (50.8, 67.9), turned to 180 degrees
- moved R25 152.9 mm to (75.6, 61.0), turned to 270 degrees
- moved C102 150.6 mm to (44.5, 66.0)
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Connections:
- removed net N$1: C13.P$1, C4.P$1, C5.P$1, C6.P$1, C7.P$1, C8.P$1
- removed net N$2: C10.P$1, C11.P$1, U1.52
- removed net N$31: D15.P$3, R41.P$2, R89.P$2
- removed net N$32: D9.P$3, R40.P$2, R90.P$2
- removed net N$36: R14.P$1, U9.13
- removed net N$37: D7.C, R14.P$2
- removed net SPI_D+: JP1.3, U9.3
- removed net SPI_D-: JP2.3, U9.4
- removed net UART_D+: JP1.1, U$13.3
- removed net UART_D-: JP2.1, U$13.4
- new net N$105: J4.2, P8.H1, P8.H10, P8.H11, P8.H12, P8.H2, P8.H3, P8.H4, P8.H5, P8.H6, P8.H7, P8.H8, P8.H9, P8.PAD, Q9.D1, Q9.D2, Q9.D3, Q9.D4
- new net N$106: JP1.1, U9.18
- new net N$107: JP1.2
- new net N$108: JP7.1, U9.22
- new net N$109: JP5.1, U9.1
- new net N$110: JP4.1, U9.23
- new net N$111: JP3.1, U9.24
- net !CS: now also J16.1, JP7.2; no longer J16.4, U9.22
- net 12V: now also J1.1; no longer J1.P$1
- net 3.3V: now also C10.P$1, C11.P$1, C13.P$1, C4.P$1, C5.P$1, C6.P$1, C7.P$1, C8.P$1, U1.52; no longer C73.P$1, C74.P$1, C75.P$1, D7.A, R44.P$2, U$13.5, U$13.6, U$13.7
- net CP2102_RX: now also J15.2, JP2.2; no longer J15.1, U$13.20
- net CP2102_TX: now also J15.1, JP6.2; no longer J15.2, U$13.21
- net D+: now also U9.3; no longer JP1.2
- net D-: now also U9.4; no longer JP2.2
- net DCBUS: now also J2.1, J4.1, P6.H1, P6.H10, P6.H11, P6.H12, P6.H2, P6.H3, P6.H4, P6.H5, P6.H6, P6.H7, P6.H8, P6.H9, P6.PAD, P7.H1, P7.H10, P7.H11, P7.H12, P7.H2, P7.H3, P7.H4, P7.H5, P7.H6, P7.H7, P7.H8, P7.H9, P7.PAD; no longer J11.P$1, J2.P$1
- net DIR: now also D9.P$3, R40.P$2, R90.P$2
- net GND: now also J1.2, J2.2, P5.H1, P5.H10, P5.H11, P5.H12, P5.H2, P5.H3, P5.H4, P5.H5, P5.H6, P5.H7, P5.H8, P5.H9, P5.PAD; no longer C73.P$2, C74.P$2, C75.P$2, J1.P$2, J2.P$2, U$13.2, U$13.PAD
- net INT: no longer U9.18
- net MISO: now also J16.4, JP3.2; no longer J16.1, U9.24
- net MOSI: now also J16.3, JP4.2; no longer J16.2, U9.23
- net N$101: now also JP2.1, U9.21; no longer J11.P$2, Q9.D1, Q9.D2, Q9.D3, Q9.D4
- net N$63: now also U9.14; no longer U$13.14
- net N$64: now also U9.13; no longer U$13.13
- net N$68: now also JP6.1, U9.20; no longer R44.P$1, U$13.9
- net SCK: now also J16.2, JP5.2; no longer J16.3, U9.1
- net STEP: now also D15.P$3, R41.P$2, R89.P$2
- net VBUS: no longer U$13.8
Routing:
- net ENO: track 0.00 -> 112.0 mm, vias 0 -> 4
- net N$54: track 0.00 -> 69.6 mm
- net PWM_Y2_L: track 0.00 -> 59.0 mm
- net PWM_Y2_H: track 0.00 -> 54.1 mm
- net BRAKE: track 0.00 -> 50.6 mm
- net PWM_UX1_L: track 0.00 -> 46.6 mm
- net PWM_UX1_H: track 0.00 -> 38.0 mm
- net PWM_WY1_L: track 0.00 -> 36.0 mm
- net SCK: track 0.00 -> 35.5 mm, vias 0 -> 2
- net N$56: track 0.00 -> 34.7 mm
- net ADC_I0_U_PF: track 0.00 -> 34.7 mm, vias 0 -> 2
- net MISO: track 0.00 -> 34.6 mm, vias 0 -> 3
- net N$55: track 0.00 -> 34.6 mm
- net CP2102_RX: track 0.00 -> 31.4 mm, vias 0 -> 2
- net CP2102_TX: track 0.00 -> 31.1 mm, vias 0 -> 2
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- added copper zone on layer 16, net GND
- added copper zone on layer 1, net N$105
- removed copper zone on layer 1, net DCBUS2
- removed copper zone on layer 1, net DCBUS3
Other:
- board size 100 x 100 mm -> 120 x 100 mm
