File: hardware/v0a/v0a.sch (EAGLE design)
At the start: 232 parts, among them J1 2EDG-2P, J2 2EDG-2P, J3 2EDG-2P, J4 2EDG-2P, J5 SH-5, J6 SH-5, J7 SH-5, J8 SH-5, J9 SH-2, Q1 IRF7580, Q2 IRF7580, Q3 IRF7580, Q4 IRF7580, Q5 IRF7580, Q6 IRF7580, Q7 IRF7580, Q8 IRF7580, U1 TMC4671, U10 AD8418, U11 AD8418, U12 DSC1101, U13 74LVC3G17, U14 74LVC3G17, U15 74LVC3G17, U16 74LVC3G17, U2 MIC39101, U3 MIC39101, U4 SI82397, U5 SI82397, U6 SI82397, U7 SI82397, U8 MIC4682, U9 CP2130

Commit message: etc
Parts:
- removed C16, C17: 100u, Passive Components > Capacitors > Aluminium Electrolytic Capacitors:CAPACITOR_EL10X10
- removed C32, C33: (no value), Passive Components > Capacitors > Tantalum Capacitors:CAPACITOR_TAN3216
- removed C46, C53, C60: 100n, Passive Components > Capacitors > Multilayer Ceramic Capacitors MLCC:MLCC0603
- removed C65: 10u, Passive Components > Capacitors > Tantalum Capacitors:CAPACITOR_TAN3216
- removed C72: 1u, Passive Components > Capacitors > Tantalum Capacitors:CAPACITOR_TAN3216
- removed U$12: USB-SHIELD, Connectors > USB:USB-SHIELD
- added C104, C105, C106, C107: (no value), Passive Components > Capacitors > Multilayer Ceramic Capacitors MLCC:MLCC0603
- added D12, D13, D14, D15, D16: BAT54S, Semiconductors > Discrete Semiconductors > Diodes & Rectifiers > Schottky Diodes & Rectifiers:BAT54S
- added D17, D18, D19: (no value), Opto-electronics > LED Emitters:LED0603
- added J10: SH-5, Connectors > JST > SH:SH-5
- added J11: 2EDG-2P, Connectors > Other:2EDG-2P
- added J12, J15: SH-3, Connectors > JST > SH:SH-3
- added J13: SH-2, Connectors > JST > SH:SH-2
- added J14: F20F-10DP-1V, Connectors > Other:F20F-10DP-1V
- added J16: SH-6, Connectors > JST > SH:SH-6
- added JP1, JP2: JUMPER-SMT_3_1-NC_PASTE_SILK, Utility > Board:JUMPER-SMT_3_1-NC_PASTE_SILK
- added Q9: IRF7580, Semiconductors > Discrete Semiconductors > Transistors > MOSFETs:IRF7580
- added R78, R79, R80, R81, R82, R83: 10k, Passive Components > Resistors > Chip Resistors:RESISTOR0603
- added R84, R85, R86: (no value), Passive Components > Resistors > Chip Resistors:RESISTOR0603
- added R87: 2.2, Passive Components > Resistors > Chip Resistors:RESISTOR0603
- added R88: 220, Passive Components > Resistors > Chip Resistors:RESISTOR0603
- added R89, R90, R91, R92: 24k, Passive Components > Resistors > Chip Resistors:RESISTOR0603
- added R93: 2k, Passive Components > Resistors > Chip Resistors:RESISTOR0603
- added R94, R95: 1k, Passive Components > Resistors > Chip Resistors:RESISTOR0603
- added U17: SI8261, Power > Gate Drivers:SI8261
- C12, C13, C14, C15, C21, C26, C30, C36, C75: device Passive Components > Capacitors > Tantalum Capacitors:CAPACITOR_TAN3216 -> Passive Components > Capacitors > Multilayer Ceramic Capacitors MLCC:MLCC0603
- C18, C20: device Passive Components > Capacitors > Aluminium Electrolytic Capacitors:CAPACITOR_EL10X10 -> Passive Components > Capacitors > Aluminium Electrolytic Capacitors:CAPACITOR_ELD
- C19: value 100u -> 10u 25v; device Passive Components > Capacitors > Aluminium Electrolytic Capacitors:CAPACITOR_EL10X10 -> Passive Components > Capacitors > Multilayer Ceramic Capacitors MLCC:MLCC0603
- C22, C23, C24, C25: value (none) -> 330u; device Passive Components > Capacitors > Aluminium Electrolytic Capacitors:CAPACITOR_EL10X10 -> Passive Components > Capacitors > Aluminium Electrolytic Capacitors:CAPACITOR_ELG
- C27: value 1u -> 100n 25v; device Passive Components > Capacitors > Tantalum Capacitors:CAPACITOR_TAN3216 -> Passive Components > Capacitors > Multilayer Ceramic Capacitors MLCC:MLCC0603
- C34, C35, C37, C38: value 220n 60v -> 220n 25v
- C39: value (none) -> 10u 25v
- C40, C41, C42, C67, C68: value (none) -> 100n
- C43, C44: value (none) -> 10u 25v; device Passive Components > Capacitors > Tantalum Capacitors:CAPACITOR_TAN3216 -> Passive Components > Capacitors > Multilayer Ceramic Capacitors MLCC:MLCC0603
- C45: value (none) -> 4u7; device Passive Components > Capacitors > Tantalum Capacitors:CAPACITOR_TAN3216 -> Passive Components > Capacitors > Multilayer Ceramic Capacitors MLCC:MLCC0603
- C48, C49, C55, C56, C62, C63: value 100n -> 100n 25v
- C50, C51, C57, C58, C64: value 10u -> 10u 25v; device Passive Components > Capacitors > Tantalum Capacitors:CAPACITOR_TAN3216 -> Passive Components > Capacitors > Multilayer Ceramic Capacitors MLCC:MLCC0603
- C52, C59, C66: value 10u -> 4u7; device Passive Components > Capacitors > Tantalum Capacitors:CAPACITOR_TAN3216 -> Passive Components > Capacitors > Multilayer Ceramic Capacitors MLCC:MLCC0603
- C76, C77: value (none) -> 100p
- D7: value SML-D12 -> (none); device Opto-electronics > LED Emitters:SML-D12 -> Opto-electronics > LED Emitters:LED0603
- D9: value SP0503BAHT -> BAT54S; device Circuit Protection > ESD Suppressors \ TVS Diodes:SP0503BAHT -> Semiconductors > Discrete Semiconductors > Diodes & Rectifiers > Schottky Diodes & Rectifiers:BAT54S
- L2: device Passive Components > Inductors, Chokes & Coils:INDUCTOR1207 -> Passive Components > Inductors, Chokes & Coils:INDUCTORCDRH104R
- R41: value 47k -> 24k
- R45, R46, R47: value (none) -> 10k
- R58: value 3.01k -> 4.2k
- renumbered U$15 to U19, U$16 to U18, U$17 to U20, U$18 to U21
Connections:
- net N$10 renamed VX2
- net N$6 renamed UX1
- removed net N$14: C37.P$2, J4-1.S, Q5.S1, Q6.D1, U6.GNDA@14
- removed net N$18: C38.P$2, J4-2.S, Q7.S1, Q8.D1, U7.GNDA@14
- new net AENC_UX_P: C104.P$1, D12.3, R84.P$2, U1-SENSO.AENC_UX_POS@25
- new net AENC_VN_P: C105.P$1, D13.3, R85.P$2, U1-SENSO.AENC_VN_POS@27
- new net AENC_WY_P: C106.P$1, D14.3, R86.P$2, U1-SENSO.AENC_WY_POS@29
- new net D+: D5.3, JP1.2, U$10.D+
- new net D-: D5.2, JP2.2, U$10.D-
- new net N$100: R88.P$1, U17.AN@2
- new net N$101: J11.2.S, Q9.D1
- new net N$102: Q9.G1, R87.P$2
- new net N$103: R87.P$1, U17.VO@6, U17.VO@7
- new net N$104: D18.AN, R95.P$1, U3.FLG
- new net N$94: R78.P$1, R79.P$2, U1-SENSO.AENC_WY_NEG@30
- new net N$95: R80.P$1, R81.P$2, U1-SENSO.AENC_VN_NEG@28
- new net N$96: R82.P$1, R83.P$2, U1-SENSO.AENC_UX_NEG@26
- new net N$97: J10.4.S, R86.P$1
- new net N$98: J10.3.S, R85.P$1
- new net N$99: J10.2.S, R84.P$1
- new net SPI_D+: JP1.3, U9.D+@3
- new net SPI_D-: JP2.3, U9.D-@4
- new net UART_D+: JP1.1, U$13.D+@3
- new net UART_D-: JP2.1, U$13.D-@4
- new net VBUS: R12.P$2, R13.P$1, U$13.VBUS@8, U9.VBUS@8
- new net WY1: C37.P$2, J4.1.S, Q5.S1, Q6.D1, U6.GNDA@14
- new net Y2: C38.P$2, J4.2.S, Q7.S1, Q8.D1, U7.GNDA@14
- net !CS: now also J16.4.S
- net 12V: now also C19.P$1, C21.P$1, C27.P$1, C39.P$1, C43.P$1, C44.P$1, C50.P$1, C51.P$1, C57.P$1, C58.P$1, C64.P$1, D19.AN, J1.1.S, U17.VDD@8; no longer C19.AN, C21.AN, C43.AN, C44.AN, C50.AN, C51.AN, C57.AN, C58.AN, C64.AN, C65.AN, J1-1.S
- net 3.3V: now also C14.P$1, C30.P$1, C45.P$1, C52.P$1, C59.P$1, C66.P$1, C75.P$1, D15.2, D16.2, D9.2, J14.1.S, U$13.VDD@6, U$13.VIO@5, U$13.VREGIN@7; no longer C14.AN, C17.AN, C27.AN, C30.AN, C39.P$1, C45.AN, C46.P$1, C52.AN, C53.P$1, C59.AN, C60.P$1, C66.AN, C72.AN, C75.AN
- net 5V: now also C107.P$1, C12.P$1, C15.P$1, D12.2, D13.2, D14.2, J10.1.S, J5.1.S, J6.1.S, J7.1.S, J8.1.S, J9.1.S, R78.P$2, R80.P$2, R82.P$2; no longer C12.AN, C15.AN, C16.AN, J5-1.S, J6-1.S, J7-1.S, J8-1.S, J9-1.S
- net ADC_T_MOSFETS: now also C77.P$1; no longer C77.P$2
- net ADC_T_MOTOR: now also C76.P$1, J9.2.S; no longer C76.P$2, J9-2.S
- net BRAKE: now also R88.P$2
- net CP2102_RX: now also J15.1.S
- net CP2102_TX: now also J15.2.S
- net DBG_SPI_MISO: now also J14.9.S
- net DBG_SPI_MOSI: now also J14.7.S
- net DBG_SPI_NSCS: now also J14.3.S
- net DBG_SPI_SCK: now also J14.5.S
- net DBG_SPI_TRG: now also J14.4.S
- net DCBUS: now also J11.1.S, J2.1.S; no longer C32.AN, C33.AN, J2-1.S
- net GND: now also C104.P$2, C105.P$2, C106.P$2, C107.P$2, C12.P$2, C13.P$2, C14.P$2, C15.P$2, C19.P$2, C21.P$2, C26.P$2, C27.P$2, C30.P$2, C36.P$2, C43.P$2, C44.P$2, C45.P$2, C50.P$2, C51.P$2, C52.P$2, C57.P$2, C58.P$2, C59.P$2, C64.P$2, C66.P$2, C75.P$2, C76.P$2, C77.P$2, D12.1, D13.1, D14.1, D15.1, D16.1, D17.CA, D18.CA, J1.2.S, J10.6.S, J10.TAB.S, J12.3.S, J12.TAB.S, J13.2.S, J13.TAB.S, J14.10.S, J14.6.S, J14.8.S, J14.TAB.S, J15.3.S, J15.TAB.S, J16.6.S, J16.TAB.S, J2.2.S, J5.6.S, J5.TAB.S, J6.6.S, J6.TAB.S, J7.6.S, J7.TAB.S, J8.6.S, J8.TAB.S, J9.TAB.S, Q9.S1, R79.P$1, R81.P$1, R83.P$1, R89.P$1, R90.P$1, R92.P$1, R93.P$1, U$13.GND@2, U$13.GND@PAD, U17.CA@3, U17.GNB@5; no longer C12.CA, C13.CA, C14.CA, C15.CA, C16.CA, C17.CA, C19.CA, C21.CA, C26.CA, C27.CA, C30.CA, C32.CA, C33.CA, C36.CA, C43.CA, C44.CA, C45.CA, C46.P$2, C50.CA, C51.CA, C52.CA, C53.P$2, C57.CA, C58.CA, C59.CA, C60.P$2, C64.CA, C65.CA, C66.CA, C72.CA, C75.CA, C76.P$1, C77.P$1, J1-2.S, J2-2.S, J5-5.S, J5-CASE.S, J6-5.S, J6-CASE.S, J7-5.S, J7-CASE.S, J8-5.S, J8-CASE.S, J9-CASE.S, R41.P$2, U$12.CASE, U$12.GND
- net INT: now also J16.5.S
- net MISO: now also J16.1.S
- net MOSI: now also J16.2.S
- net N$1: now also C13.P$1; no longer C13.AN
- net N$11: now also D2.C
- net N$28: now also J3.2.S; no longer J3-2.S
- net N$29: now also J3.1.S; no longer J3-1.S
- net N$31: now also D15.3, R41.P$2, R89.P$2; no longer D5.3, U$10.D+, U9.D+@3
- net N$32: now also D9.3, R40.P$2, R90.P$2; no longer D5.2, U$10.D-, U9.D-@4
- net N$33: now also J12.2.S, R41.P$1; no longer R12.P$2, R13.P$1, U9.VBUS@8
- net N$35: now also C26.P$1; no longer C26.AN
- net N$5: now also C36.P$1, R94.P$2, R95.P$2; no longer C36.AN
- net N$59: now also J12.1.S; no longer D9.4, U$12.VBUS
- net N$60: now also D17.AN, R94.P$1, U2.FLG; no longer D9.3, U$12.D+, U$13.D+@3
- net N$61: now also J13.1.S, R91.P$1; no longer D9.2, U$12.D-, U$13.D-@4
- net N$62: now also D19.CA, R93.P$2; no longer R40.P$2, R41.P$1, U$13.VBUS@8
- net N$71: now also J5.2.S; no longer J5-2.S
- net N$72: now also J5.3.S; no longer J5-3.S
- net N$73: now also J5.4.S; no longer J5-4.S
- net N$76: now also J6.2.S; no longer J6-2.S
- net N$77: now also J6.3.S; no longer J6-3.S
- net N$78: now also J6.4.S; no longer J6-4.S
- net N$82: now also J7.2.S; no longer J7-2.S
- net N$83: now also J7.3.S; no longer J7-3.S
- net N$84: now also J7.4.S; no longer J7-4.S
- net N$88: now also J8.2.S; no longer J8-2.S
- net N$89: now also J8.3.S; no longer J8-3.S
- net N$90: now also J8.4.S; no longer J8-4.S
- net PWM_IN: now also D16.3, R91.P$2, R92.P$2
- net SCK: now also J16.3.S
Other:
- note added: "Vo = 1.23 * (R3/R4 + 1) Vo ~ 5.5V"
- note removed: "Vo = 1.23 * (R3/R4 + 1) Vo ~ 4.31V"

Commit message: pcb work
Parts:
- removed J4: 2EDG-2P, Connectors > Other:2EDG-2P
- added C16, C17, C32, C33, C46, C53: 100n, Passive Components > Capacitors > Multilayer Ceramic Capacitors MLCC:MLCC0603
- added P1, P2, P3, P4: POWPAD, Connectors > Other:POWPAD
- added R96, R97, R98, R99: (no value), Passive Components > Resistors > Chip Resistors:RESISTOR0603
- D1, D2, D3, D4: value SK54L -> DSK24; device Semiconductors > Discrete Semiconductors > Diodes & Rectifiers > Schottky Diodes & Rectifiers:SK54L -> Semiconductors > Discrete Semiconductors > Diodes & Rectifiers > Schottky Diodes & Rectifiers:DSK24
- J3: value 2EDG-2P -> 4P-6.35P; device Connectors > Other:2EDG-2P -> Connectors > Other:4P-6.35P
- U10, U11: value AD8418 -> AD8418A; device Semiconductors > Integrated Circuits - ICs > Amplifier ICs > Current Sense Amplifiers:AD8418 -> Semiconductors > Integrated Circuits - ICs > Amplifier ICs > Current Sense Amplifiers:AD8418A
Connections:
- new net N$10: R9.SENSE-, R96.P$1
- new net N$14: C16.P$1, C17.P$2, R96.P$2, U10_.IN-@1
- new net N$18: C16.P$2, C32.P$1, R97.P$2, U10_.IN+@8
- new net N$6: R9.SENSE+, R97.P$1
- net GND: now also C17.P$1, C32.P$2, C46.P$1, C53.P$2
- net N$28: now also P2.S
- net N$29: now also P1.S
- net N$55: now also R98.P$1; no longer U11_.IN-@1
- net N$56: now also R99.P$1; no longer U11_.IN+@8
- net N$57: now also C33.P$2, C53.P$1, R99.P$2, U11_.IN+@8; no longer R9.SENSE-, U10_.IN-@1
- net N$58: now also C33.P$1, C46.P$2, R98.P$2, U11_.IN-@1; no longer R9.SENSE+, U10_.IN+@8
- net WY1: now also J3.3.S, P3.S; no longer J4.1.S
- net Y2: now also J3.4.S, P4.S; no longer J4.2.S
Other:
- moved on the sheet: C67, C68, J3.1, J3.2, R10, R9, U10-GND, U10-VDD, U10-VREF1, U10-VREF2, U10_, U11-GND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

Commit message: pcb work
Parts:
- removed C73, C74: 100n, Passive Components > Capacitors > Multilayer Ceramic Capacitors MLCC:MLCC0603
- removed C75: 4u7, Passive Components > Capacitors > Multilayer Ceramic Capacitors MLCC:MLCC0603
- removed D7: (no value), Opto-electronics > LED Emitters:LED0603
- removed J11: 2EDG-2P, Connectors > Other:2EDG-2P
- removed R14: 10k, Passive Components > Resistors > Chip Resistors:RESISTOR0603
- removed R44: (no value), Passive Components > Resistors > Chip Resistors:RESISTOR0603
- added J4: 2P-6.35P, Connectors > Other:2P-6.35P
- added JP3, JP4, JP5, JP7: JUMPER-SMT_2_NC_PASTE_SILK, Utility > Board:JUMPER-SMT_2_NC_PASTE_SILK
- added JP6: JUMPER-SMT_2_NO_SILK, Utility > Board:JUMPER-SMT_2_NO_SILK
- added P5, P6, P7, P8: POWPAD, Connectors > Other:POWPAD
- added U$12, U$15, U$16: MOUNTINGHOLE3.0, Utility > Board:MOUNTINGHOLE3.0
- J1, J2: value 2EDG-2P -> 2P-6.35P; device Connectors > Other:2EDG-2P -> Connectors > Other:2P-6.35P
- JP1: value JUMPER-SMT_3_1-NC_PASTE_SILK -> JUMPER-SMT_2_NC_PASTE_SILK; device Utility > Board:JUMPER-SMT_3_1-NC_PASTE_SILK -> Utility > Board:JUMPER-SMT_2_NC_PASTE_SILK
- JP2: value JUMPER-SMT_3_1-NC_PASTE_SILK -> JUMPER-SMT_2_NO_SILK; device Utility > Board:JUMPER-SMT_3_1-NC_PASTE_SILK -> Utility > Board:JUMPER-SMT_2_NO_SILK
- U$13: value CP2102N -> MOUNTINGHOLE3.0; device Semiconductors > Integrated Circuits - ICs > Interface ICs > USB Interface IC:CP2102N -> Utility > Board:MOUNTINGHOLE3.0
- U9: value CP2130 -> CP2130/2102N; device Semiconductors > Integrated Circuits - ICs > Interface ICs > USB Interface IC:CP2130 -> Semiconductors > Integrated Circuits - ICs > Interface ICs > USB Interface IC:CP2130/2102N
Connections:
- removed net N$1: C13.P$1, C4.P$1, C5.P$1, C6.P$1, C7.P$1, C8.P$1
- removed net N$2: C10.P$1, C11.P$1, U1-POW.PLL_VCC@52
- removed net N$31: D15.3, R41.P$2, R89.P$2
- removed net N$32: D9.3, R40.P$2, R90.P$2
- removed net N$36: R14.P$1, U9.GPIO8-!CS8!-SPIACT@13
- removed net N$37: D7.CA, R14.P$2
- removed net SPI_D+: JP1.3, U9.D+@3
- removed net SPI_D-: JP2.3, U9.D-@4
- removed net UART_D+: JP1.1, U$13.D+@3
- removed net UART_D-: JP2.1, U$13.D-@4
- new net N$105: J4.2.S, P8.S, Q9.D1
- new net N$106: JP1.1, U9.(CTS)GPIO4-!CS4!-EVTCNTR@18
- new net N$107: JP1.2
- new net N$108: JP7.1, U9.(DSR)GPIO0-!CS0@22
- new net N$109: JP5.1, U9.(RI/CLK)SCK@1
- new net N$110: JP4.1, U9.(DTR)MOSI@23
- new net N$111: JP3.1, U9.(DCD)MISO@24
- net !CS: now also J16.1.S, JP7.2; no longer J16.4.S, U9.GPIO0-!CS0@22
- net 3.3V: now also C10.P$1, C11.P$1, C13.P$1, C4.P$1, C5.P$1, C6.P$1, C7.P$1, C8.P$1, U1-POW.PLL_VCC@52; no longer C73.P$1, C74.P$1, C75.P$1, D7.AN, R44.P$2, U$13.VDD@6, U$13.VIO@5, U$13.VREGIN@7
- net CP2102_RX: now also J15.2.S, JP2.2; no longer J15.1.S, U$13.RXD@20
- net CP2102_TX: now also J15.1.S, JP6.2; no longer J15.2.S, U$13.TXD@21
- net D+: now also U9.D+@3; no longer JP1.2
- net D-: now also U9.D-@4; no longer JP2.2
- net DCBUS: now also J4.1.S, P6.S, P7.S; no longer J11.1.S
- net DIR: now also D9.3, R40.P$2, R90.P$2
- net GND: now also P5.S; no longer C73.P$2, C74.P$2, C75.P$2, U$13.GND@2, U$13.GND@PAD
- net INT: no longer U9.GPIO4-!CS4!-EVTCNTR@18
- net MISO: now also J16.4.S, JP3.2; no longer J16.1.S, U9.MISO@24
- net MOSI: now also J16.3.S, JP4.2; no longer J16.2.S, U9.MOSI@23
- net N$101: now also JP2.1, U9.(TXD)GPIO1-!CS1@21; no longer J11.2.S, Q9.D1
- net N$63: now also U9.(GPIO0-TXT)GPIO7-!CS7@14; no longer U$13.GPIO0-TXT@14
- net N$64: now also U9.(GPIO1-RXT)GPIO8-!CS8!-SPIACT@13; no longer U$13.GPIO1-RXT@13
- net N$68: now also JP6.1, U9.(RXD)GPIO2-!CS2@20; no longer R44.P$1, U$13.RSTB@9
- net SCK: now also J16.2.S, JP5.2; no longer J16.3.S, U9.SCK@1
- net STEP: now also D15.3, R41.P$2, R89.P$2
- net VBUS: no longer U$13.VBUS@8
Other:
- moved on the sheet: C26, C28, C29, C30, D10, D11, J15.1, J15.2, J15.3, J15.TAB, R11, R42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
