File: hardware/v0a/servo-ctrl.sch (EAGLE design)
At the start: 282 parts, among them J1 2P-6.35P, J10 SH-5, J12 SH-3, J13 SH-2, J14 F20F-10DP-1V, J15 SH-3, J16 SH-6, J2 2P-6.35P, J3 4P-6.35P, J4 2P-6.35P, J5 SH-5, J6 SH-5, J7 SH-5, J8 SH-5, J9 SH-2, P1 POWPAD, P2 POWPAD, P3 POWPAD, P4 POWPAD, P5 POWPAD, P6 POWPAD, P7 POWPAD, P8 POWPAD, Q1 IRF7580, Q2 IRF7580, Q3 IRF7580, Q4 IRF7580, Q5 IRF7580, Q6 IRF7580, Q7 IRF7580, Q8 IRF7580, Q9 IRF7580, U1 TMC4671, U10 AD8418A, U11 AD8418A, U12 DSC1101, U13 74LVC3G17, U14 74LVC3G17, U15 74LVC3G17, U16 74LVC3G17, U17 SI8261, U18 SRV05-4, U19 SRV05-4, U2 MIC39101, U20 SRV05-4, U21 SRV05-4, U3 MIC39101, U4 SI82397, U5 SI82397, U6 SI82397, U7 SI82397, U8 MIC4682, U9 CP2130/2102N

Commit message: pcb 80% finished
Parts:
- removed C1, C13, C2, C3, C31, C4, C5, C6, C7: (no value), Passive Components > Capacitors > Multilayer Ceramic Capacitors MLCC:MLCC0603
- removed C19, C39, C43, C44, C50, C51, C57, C58, C64: 10u 25v, Passive Components > Capacitors > Multilayer Ceramic Capacitors MLCC:MLCC0603
- removed C27: 100n 25v, Passive Components > Capacitors > Multilayer Ceramic Capacitors MLCC:MLCC0603
- removed C30: 4u7, Passive Components > Capacitors > Multilayer Ceramic Capacitors MLCC:MLCC0603
- removed C33, C46, C53, C68: 100n, Passive Components > Capacitors > Multilayer Ceramic Capacitors MLCC:MLCC0603
- removed D18, D19: (no value), Opto-electronics > LED Emitters:LED0603
- removed J1, J4: 2P-6.35P, Connectors > Other:2P-6.35P
- removed P2, P3, P7, P8: POWPAD, Connectors > Other:POWPAD
- removed Q9: IRF7580, Semiconductors > Discrete Semiconductors > Transistors > MOSFETs:IRF7580
- removed R10: 700u, Passive Components > Resistors > Current Sense:LRMAP3920
- removed R87: 2.2, Passive Components > Resistors > Chip Resistors:RESISTOR0603
- removed R88: 220, Passive Components > Resistors > Chip Resistors:RESISTOR0603
- removed R93: 2k, Passive Components > Resistors > Chip Resistors:RESISTOR0603
- removed R95: 1k, Passive Components > Resistors > Chip Resistors:RESISTOR0603
- removed R98, R99: (no value), Passive Components > Resistors > Chip Resistors:RESISTOR0603
- removed U$12, U$13, U$15, U$16: MOUNTINGHOLE3.0, Utility > Board:MOUNTINGHOLE3.0
- removed U11: AD8418A, Semiconductors > Integrated Circuits - ICs > Amplifier ICs > Current Sense Amplifiers:AD8418A
- removed U17: SI8261, Power > Gate Drivers:SI8261
- added C108, C217, C423, C429, C430, C431: 100n, Passive Components > Capacitors > Multilayer Ceramic Capacitors MLCC:MLCC0603
- added C114, C115, C226, C227, C228: 100p, Passive Components > Capacitors > Multilayer Ceramic Capacitors MLCC:MLCC0603
- added C205: 4u7, Passive Components > Capacitors > Multilayer Ceramic Capacitors MLCC:MLCC0603
- added C421: 100n 25v, Passive Components > Capacitors > Multilayer Ceramic Capacitors MLCC:MLCC0603
- added C424: 10u 25v, Passive Components > Capacitors > Multilayer Ceramic Capacitors MLCC:MLCC0603
- added J301, J403: 2P-6.35P, Connectors > Other:2P-6.35P
- added P401, P404, P405, P406: POWPAD, Connectors > Other:POWPAD
- added Q409: IRF7580, Semiconductors > Discrete Semiconductors > Transistors > MOSFETs:IRF7580
- added R422: 700u, Passive Components > Resistors > Current Sense:LRMAP3920
- added R425, R426: 100, Passive Components > Resistors > Chip Resistors:RESISTOR0603
- added R429: 220, Passive Components > Resistors > Chip Resistors:RESISTOR0603
- added R431: 2.2, Passive Components > Resistors > Chip Resistors:RESISTOR0603
- added U406: AD8418A, Semiconductors > Integrated Circuits - ICs > Amplifier ICs > Current Sense Amplifiers:AD8418A
- added U407: SI8261, Power > Gate Drivers:SI8261
- C102, C103: value 100p -> 100n
- C104, C105, C106, C107, C109: value (none) -> 100n
- C201, C203, C204: value (none) -> 4u7
- C202: value 1u -> 4u7
- C206, C207, C208, C209, C210, C211, C212, C213, C218, C219, C220, C221: value (none) -> 100p
- C406: value 100n -> 10u 25v
- C408, C410, C412: value 100n 25v -> 10u 25v
- C502: value 100n -> 4u7
- D302, D501, D502: value (none) -> LED0603
- R101, R102: value (none) -> 10k
- R201, R202, R203, R204, R205, R206, R207, R208, R209, R210, R211, R212, R213, R218, R227, R423, R424: value (none) -> 100
- R305: value 1k -> 2k
- R427: value 10k -> 100k
- R428: value 10k -> 1k13
- R502, R503: value (none) -> 220
- renumbered C10 to C110, C100 to C225, C11 to C111, C12 to C113, C14 to C309, C15 to C310, C16 to C427, C17 to C426, C18 to C307, C20 to C302, C21 to C301, C22 to C303, C23 to C304, C24 to C306, C25 to C308, C26 to C503, C28 to C502, C29 to C501, C32 to C428, C34 to C417, C35 to C418, C36 to C305, C37 to C419, C38 to C420, C40 to C413, C41 to C401, C42 to C406, C45 to C405, C47 to C414, C48 to C402, C49 to C408, C52 to C407, C54 to C415, C55 to C403, C56 to C410, C59 to C409, C61 to C416, C62 to C404, C63 to C412, C66 to C411, C67 to C422, C69 to C116, C70 to C117, C71 to C118, C76 to C432, C77 to C425, C78 to C206, C79 to C210, C8 to C109, C80 to C218, C81 to C201, C82 to C207, C83 to C211, C84 to C219, C85 to C202, C86 to C208, C87 to C212, C88 to C220, C89 to C203, C9 to C112, C90 to C222, C91 to C223, C92 to C215, C93 to C224, C94 to C216, C95 to C214, C96 to C209, C97 to C213, C98 to C221, C99 to C204, D1 to D401, D10 to D502, D11 to D501, D12 to D201, D13 to D202, D14 to D203, D15 to D506, D16 to D504, D17 to D302, D2 to D402, D3 to D403, D4 to D404, D5 to D503, D6 to D301, D8 to D101, D9 to D505, J10 to J205, J12 to J506, J13 to J504, J14 to J505, J15 to J502, J16 to J501, J2 to J302, J3 to J401, J5 to J201, J6 to J202, J7 to J203, J8 to J204, J9 to J402, JP1 to JP507, JP2 to JP505, JP3 to JP501, JP4 to JP502, JP5 to JP503, JP6 to JP506, JP7 to JP504, L2 to L301, P1 to P403, P4 to P402, P5 to P302, P6 to P301, Q1 to Q401, Q2 to Q405, Q3 to Q402, Q4 to Q406, Q5 to Q403, Q6 to Q407, Q7 to Q404, Q8 to Q408, R1 to R413, R11 to R501, R12 to R506, R13 to R507, R15 to R108, R16 to R105, R17 to R405, R18 to R401, R19 to R406, R2 to R417, R20 to R402, R21 to R407, R22 to R403, R23 to R408, R24 to R404, R25 to R101, R26 to R114, R27 to R102, R28 to R409, R29 to R410, R3 to R414, R30 to R411, R31 to R412, R32 to R117, R33 to R118, R34 to R120, R35 to R121, R36 to R113, R37 to R115, R38 to R119, R39 to R116, R4 to R418, R40 to R508, R41 to R509, R42 to R502, R43 to R503, R45 to R428, R46 to R430, R47 to R427, R48 to R201, R49 to R202, R5 to R415, R50 to R203, R51 to R204, R52 to R205, R53 to R206, R54 to R207, R55 to R301, R56 to R302, R57 to R208, R58 to R303, R59 to R304, R6 to R419, R60 to R209, R61 to R216, R62 to R221, R63 to R225, R64 to R215, R65 to R220, R66 to R224, R67 to R214, R68 to R219, R69 to R223, R7 to R416, R70 to R210, R71 to R211, R72 to R212, R73 to R217, R74 to R222, R75 to R226, R76 to R111, R77 to R112, R78 to R109, R79 to R110, R8 to R420, R80 to R106, R81 to R107, R82 to R103, R83 to R104, R84 to R213, R85 to R218, R86 to R227, R89 to R510, R9 to R421, R90 to R511, R91 to R504, R92 to R505, R94 to R305, R96 to R423, R97 to R424, U$10 to J503, U1 to U102, U10 to U405, U12 to U101, U13 to U205, U14 to U206, U15 to U207, U16 to U208, U18 to U202, U19 to U201, U2 to U302, U20 to U203, U21 to U204, U3 to U303, U4 to U401, U5 to U402, U6 to U403, U7 to U404, U8 to U301, U9 to U501
Connections:
- removed net GPIO0: U102-IO.GPIO0@70
- removed net GPIO1: U102-IO.GPIO1@71
- removed net GPIO2: U102-IO.GPIO2@74
- removed net N$107: JP507.2
- removed net N$28: J401.2.S, P2.S, R10.P$2
- removed net N$60: D302.AN, R305.P$1, U302.FLG
- removed net N$62: D19.CA, R93.P$2
- new net N$1: J401.3.S, P404.S, R422.P$2
- net 1.8V: now also C103.P$1, C105.P$1, C107.P$1; no longer C1.P$1, C2.P$1, C3.P$1
- net 12V: now also C421.P$1, C424.P$1, J301.2.S, U407.VDD@8; no longer C19.P$1, C27.P$1, C39.P$1, C43.P$1, C44.P$1, C50.P$1, C51.P$1, C57.P$1, C58.P$1, C64.P$1, D19.AN, J1.1.S, U17.VDD@8
- net 3.3V: now also C102.P$1, C104.P$1, C106.P$1, C108.P$1, C217.P$1; no longer C13.P$1, C30.P$1, C31.P$1, C4.P$1, C5.P$1, C6.P$1, C7.P$1
- net 5V: now also C205.P$1, C423.P$1, U406-VDD.P$1, U406-VREF1.P$1; no longer C107.P$1, C68.P$1, U11-VDD.P$1, U11-VREF1.P$1
- net ADC_I1_V_PF: now also U406_.O@5; no longer U11_.O@5
- net AENC_UX_P: now also C226.P$1; no longer C104.P$1
- net AENC_VN_P: now also C227.P$1; no longer C105.P$1
- net AENC_WY_P: now also C228.P$1; no longer C106.P$1
- net BRAKE: now also R429.P$2; no longer R88.P$2
- net DCBUS: now also J403.1.S, P405.S; no longer J4.1.S, P7.S
- net GND: now also C108.P$2, C114.P$2, C115.P$2, C205.P$2, C217.P$2, C226.P$2, C227.P$2, C228.P$2, C421.P$2, C423.P$2, C424.P$2, C429.P$1, C431.P$2, J301.1.S, Q409.S1, U406-GND.P$1, U406-VREF2.P$1, U407.CA@3, U407.GNB@5; no longer C1.P$2, C13.P$2, C19.P$2, C2.P$2, C27.P$2, C3.P$2, C30.P$2, C31.P$2, C39.P$2, C4.P$2, C43.P$2, C44.P$2, C46.P$1, C5.P$2, C50.P$2, C51.P$2, C53.P$2, C57.P$2, C58.P$2, C6.P$2, C64.P$2, C68.P$2, C7.P$2, D18.CA, J1.2.S, Q9.S1, R93.P$1, U11-GND.P$1, U11-VREF2.P$1, U17.CA@3, U17.GNB@5
- net INT: now also JP507.2
- net N$100: now also R429.P$1, U407.AN@2; no longer R88.P$1, U17.AN@2
- net N$102: now also Q409.G1, R431.P$2; no longer Q9.G1, R87.P$2
- net N$103: now also R431.P$1, U407.VO@6, U407.VO@7; no longer R87.P$1, U17.VO@6, U17.VO@7
- net N$104: now also D302.AN, R305.P$1, U302.FLG; no longer D18.AN, R95.P$1
- net N$105: now also J403.2.S, P406.S, Q409.D1; no longer J4.2.S, P8.S, Q9.D1
- net N$5: no longer R95.P$2
- net N$55: now also R422.SENSE-, R425.P$1; no longer R10.SENSE-, R98.P$1
- net N$56: now also R422.SENSE+, R426.P$1; no longer R10.SENSE+, R99.P$1
- net N$57: now also C430.P$2, C431.P$1, R426.P$2, U406_.IN+@8; no longer C33.P$2, C53.P$1, R99.P$2, U11_.IN+@8
- net N$58: now also C429.P$2, C430.P$1, R425.P$2, U406_.IN-@1; no longer C33.P$1, C46.P$2, R98.P$2, U11_.IN-@1
- net N$67: now also U201.2; no longer U201.3
- net N$69: now also U201.4; no longer U201.2
- net N$70: now also U202.2; no longer U202.3
- net N$75: now also U202.4; no longer U202.2
- net N$80: now also U203.2; no longer U203.3
- net N$81: now also U203.4; no longer U203.2
- net N$86: now also U204.2; no longer U204.3
- net N$87: now also U204.4; no longer U204.2
- net N$92: now also C114.P$1; no longer C102.P$1
- net N$93: now also C115.P$1; no longer C103.P$1
- net VX2: now also J401.2.S, P401.S; no longer R10.P$1
- net WY1: now also R422.P$1; no longer J401.3.S, P3.S
Other:
- note added: "1.24v at 125ºc"
