File: hardware/hv0a/servo-ctrl.sch (EAGLE design)
At the start: 264 parts, among them J201 SH-5, J202 SH-5, J203 SH-5, J204 SH-5, J205 SH-5, J301 2P-6.35P, J302 2P-6.35P, J401 4P-6.35P, J402 SH-2, J403 2P-6.35P, J501 SH-6, J502 SH-3, J503 USB-SHIELD, J504 SH-2, J505 F20F-10DP-1V, J506 SH-3, P301 POWPAD, P302 POWPAD, P401 POWPAD, P402 POWPAD, P403 POWPAD, P404 POWPAD, P405 POWPAD, P406 POWPAD, Q401 IRF7580, Q402 IRF7580, Q403 IRF7580, Q404 IRF7580, Q405 IRF7580, Q406 IRF7580, Q407 IRF7580, Q408 IRF7580, Q409 IRF7580, U101 DSC1101, U102 TMC4671, U201 SRV05-4, U202 SRV05-4, U203 SRV05-4, U204 SRV05-4, U205 74LVC3G17, U206 74LVC3G17, U207 74LVC3G17, U208 74LVC3G17, U301 MIC4682, U302 MIC39101, U303 MIC39101, U401 SI82397, U402 SI82397, U403 SI82397, U404 SI82397, U405 AD8418A, U406 AD8418A, U407 SI8261, U501 CP2130/2102N

Commit message: finished pcb, added pdf and png exports of pcb
Connections:
- net N$1 renamed WY1@J401
- net N$29 renamed UX1@J401
- net N$33 renamed STEP@J
- net N$59 renamed DIR@J
- net N$61 renamed PWM_IN@J
- net N$71 renamed ENC_A@J
- net N$72 renamed ENC_B@J
- net N$73 renamed ENC_N@J
- net N$76 renamed ENC_2_A@J
- net N$77 renamed ENC_2_B@J
- net N$78 renamed ENC_2_N@J
- net N$82 renamed HALL_WY@J
- net N$83 renamed HALL_V@J
- net N$84 renamed HALL_UX@J
- net N$88 renamed REF_R@J
- net N$89 renamed REF_H@J
- net N$90 renamed REF_L@J
- net N$97 renamed AENC_WY@J
- net N$98 renamed AENC_VN@J
- net N$99 renamed AENC_UX@J
Changed lines of the file:
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@@
 </segment>
 </net>
-<net name="N$71" class="0">
+<net name="ENC_A@J" class="0">
 <segment>
 <pinref part="J201" gate=".2" pin="S"/>
@@
 </segment>
 </net>
-<net name="N$72" class="0">
+<net name="ENC_B@J" class="0">
 <segment>
 <pinref part="J201" gate=".3" pin="S"/>
@@
 </segment>
 </net>
-<net name="N$73" class="0">
+<net name="ENC_N@J" class="0">
 <segment>
 <pinref part="J201" gate=".4" pin="S"/>
@@
 </segment>
 </net>
-<net name="N$76" class="0">
+<net name="ENC_2_A@J" class="0">
 <segment>
 <pinref part="J202" gate=".2" pin="S"/>
@@
 </segment>
 </net>
-<net name="N$77" class="0">
+<net name="ENC_2_B@J" class="0">
 <segment>
 <pinref part="J202" gate=".3" pin="S"/>
@@
 </segment>
 </net>
-<net name="N$78" class="0">
+<net name="ENC_2_N@J" class="0">
 <segment>
 <pinref part="J202" gate=".4" pin="S"/>
@@
 </segment>
 </net>
-<net name="N$82" class="0">
+<net name="HALL_WY@J" class="0">
 <segment>
 <pinref part="J203" gate=".2" pin="S"/>
@@
 </segment>
 </net>
-<net name="N$83" class="0">
+<net name="HALL_V@J" class="0">
 <segment>
 <pinref part="J203" gate=".3" pin="S"/>
@@
 </segment>
 </net>
-<net name="N$84" class="0">
+<net name="HALL_UX@J" class="0">
 <segment>
 <pinref part="J203" gate=".4" pin="S"/>
@@
 </segment>
 </net>
-<net name="N$88" class="0">
+<net name="REF_R@J" class="0">
 <segment>
 <pinref part="J204" gate=".2" pin="S"/>
@@
 </segment>
 </net>
-<net name="N$89" class="0">
+<net name="REF_H@J" class="0">
 <segment>
 <pinref part="J204" gate=".3" pin="S"/>
@@
 </segment>
 </net>
-<net name="N$90" class="0">
+<net name="REF_L@J" class="0">
 <segment>
 <pinref part="J204" gate=".4" pin="S"/>
@@
 </segment>
 </net>
-<net name="N$97" class="0">
+<net name="AENC_WY@J" class="0">
 <segment>
 <pinref part="J205" gate=".4" pin="S"/>
@@
 </segment>
 </net>
-<net name="N$98" class="0">
+<net name="AENC_VN@J" class="0">
 <segment>
 <pinref part="J205" gate=".3" pin="S"/>
@@
 </segment>
 </net>
-<net name="N$99" class="0">
+<net name="AENC_UX@J" class="0">
 <segment>
 <pinref part="J205" gate=".2" pin="S"/>
@@
 </segment>
 </net>
-<net name="N$29" class="0">
+<net name="UX1@J401" class="0">
 <segment>
 <pinref part="R421" gate="G$1" pin="P$2"/>
@@
 <wire x1="203.2" y1="233.68" x2="203.2" y2="236.22" width="0.1524" layer="91"/>
 <junction x="203.2" y="236.22"/>
+<label x="203.2" y="236.22" size="0.889" layer="95" rot="R180" xref="yes"/>
 </segment>
 </net>
@@
 </segment>
 </net>
-<net name="N$1" class="0">
+<net name="WY1@J401" class="0">
 <segment>
 <pinref part="R422" gate="G$1" pin="P$2"/>
@@
 <wire x1="203.2" y1="139.7" x2="203.2" y2="137.16" width="0.1524" layer="91"/>
 <junction x="203.2" y="137.16"/>
+<label x="203.2" y="137.16" size="0.889" layer="95" rot="R180" xref="yes"/>
 </segment>
 </net>
@@
 </segment>
 </net>
-<net name="N$33" class="0">
+<net name="STEP@J" class="0">
 <segment>
 <pinref part="J506" gate=".2" pin="S"/>
@@
 </segment>
 </net>
-<net name="N$59" class="0">
+<net name="DIR@J" class="0">
 <segment>
 <pinref part="J506" gate=".1" pin="S"/>
@@
 </segment>
 </net>
-<net name="N$61" class="0">
+<net name="PWM_IN@J" class="0">
 <segment>
 <pinref part="J504" gate=".1" pin="S"/>

Commit message: bom
Parts:
- C118: value 10n -> 100p
Other:
- moved on the sheet: C201, C202, C203, C204, C205, C206, C207, C208, C209, C210, C211, C212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

Commit message: component request preparation
Parts:
- C111: value 470n -> 4u7
- R428: value 1k13 -> 1k2
- R430: value 10k -> 1k2
Other:
- note added: "1.24v at 125ºc @ R428 = 1k13"
- note removed: "1.24v at 125ºc"
Changed lines of the file:
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@@
 <part name="C112" library="Passive Components &gt; Capacitors &gt; Multilayer Ceramic Capacitors MLCC" deviceset="MLCC" device="0603" value="100n"/>
 <part name="C110" library="Passive Components &gt; Capacitors &gt; Multilayer Ceramic Capacitors MLCC" deviceset="MLCC" device="0603" value="100n"/>
-<part name="C111" library="Passive Components &gt; Capacitors &gt; Multilayer Ceramic Capacitors MLCC" deviceset="MLCC" device="0603" value="470n"/>
+<part name="C111" library="Passive Components &gt; Capacitors &gt; Multilayer Ceramic Capacitors MLCC" deviceset="MLCC" device="0603" value="4u7"/>
 <part name="C113" library="Passive Components &gt; Capacitors &gt; Multilayer Ceramic Capacitors MLCC" deviceset="MLCC" device="0603" value="4u7"/>
 <part name="C109" library="Passive Components &gt; Capacitors &gt; Multilayer Ceramic Capacitors MLCC" deviceset="MLCC" device="0603" value="100n"/>
@@
 <part name="GND434" library="Utility &gt; Power Symbols" deviceset="GND" device=""/>
 <part name="SUPPLY430" library="Utility &gt; Power Symbols" deviceset="5V" device=""/>
-<part name="R428" library="Passive Components &gt; Resistors &gt; Chip Resistors" deviceset="RESISTOR" device="0603" value="1k13"/>
-<part name="R430" library="Passive Components &gt; Resistors &gt; Chip Resistors" deviceset="RESISTOR" device="0603" value="10k"/>
+<part name="R428" library="Passive Components &gt; Resistors &gt; Chip Resistors" deviceset="RESISTOR" device="0603" value="1k2"/>
+<part name="R430" library="Passive Components &gt; Resistors &gt; Chip Resistors" deviceset="RESISTOR" device="0603" value="1k2"/>
 <part name="GND442" library="Utility &gt; Power Symbols" deviceset="GND" device=""/>
 <part name="SUPPLY431" library="Utility &gt; Power Symbols" deviceset="5V" device=""/>
@@
 <wire x1="281.94" y1="147.32" x2="200.66" y2="147.32" width="0.645159375" layer="97" style="longdash"/>
 <wire x1="200.66" y1="147.32" x2="200.66" y2="193.04" width="0.645159375" layer="97" style="longdash"/>
-<text x="210.82" y="53.34" size="1.778" layer="97" rot="R90">1.24v at 125ºc</text>
+<text x="208.28" y="50.8" size="1.778" layer="97" rot="R90">1.24v at 125ºc @ R428 = 1k13</text>
 </plain>
 <instances>

Commit message: component request
Parts:
- R504, R508, R509: value 24k -> 100
- R505, R510, R511: value 24k -> 10k
- R506: value 24k -> 5k
- R507: value 47k -> 10k
Changed lines of the file:
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@@
 <part name="D503" library="Circuit Protection &gt; ESD Suppressors \ TVS Diodes" deviceset="SP0503BAHT" device=""/>
 <part name="GND509" library="Utility &gt; Power Symbols" deviceset="GND" device=""/>
-<part name="R506" library="Passive Components &gt; Resistors &gt; Chip Resistors" deviceset="RESISTOR" device="0603" value="24k"/>
-<part name="R507" library="Passive Components &gt; Resistors &gt; Chip Resistors" deviceset="RESISTOR" device="0603" value="47k"/>
+<part name="R506" library="Passive Components &gt; Resistors &gt; Chip Resistors" deviceset="RESISTOR" device="0603" value="5k"/>
+<part name="R507" library="Passive Components &gt; Resistors &gt; Chip Resistors" deviceset="RESISTOR" device="0603" value="10k"/>
 <part name="GND512" library="Utility &gt; Power Symbols" deviceset="GND" device=""/>
 <part name="D505" library="Semiconductors &gt; Discrete Semiconductors &gt; Diodes &amp; Rectifiers &gt; Schottky Diodes &amp; Rectifiers" deviceset="BAT54S" device=""/>
@@
 <part name="J506" library="Connectors &gt; JST &gt; SH" deviceset="SH-3" device=""/>
 <part name="J504" library="Connectors &gt; JST &gt; SH" deviceset="SH-2" device=""/>
-<part name="R508" library="Passive Components &gt; Resistors &gt; Chip Resistors" deviceset="RESISTOR" device="0603" value="24k"/>
-<part name="R509" library="Passive Components &gt; Resistors &gt; Chip Resistors" deviceset="RESISTOR" device="0603" value="24k"/>
+<part name="R508" library="Passive Components &gt; Resistors &gt; Chip Resistors" deviceset="RESISTOR" device="0603" value="100"/>
+<part name="R509" library="Passive Components &gt; Resistors &gt; Chip Resistors" deviceset="RESISTOR" device="0603" value="100"/>
 <part name="GND513" library="Utility &gt; Power Symbols" deviceset="GND" device=""/>
 <part name="GND514" library="Utility &gt; Power Symbols" deviceset="GND" device=""/>
@@
 <part name="SUPPLY508" library="Utility &gt; Power Symbols" deviceset="3.3V" device=""/>
 <part name="GND507" library="Utility &gt; Power Symbols" deviceset="GND" device=""/>
-<part name="R504" library="Passive Components &gt; Resistors &gt; Chip Resistors" deviceset="RESISTOR" device="0603" value="24k"/>
-<part name="R505" library="Passive Components &gt; Resistors &gt; Chip Resistors" deviceset="RESISTOR" device="0603" value="24k"/>
-<part name="R510" library="Passive Components &gt; Resistors &gt; Chip Resistors" deviceset="RESISTOR" device="0603" value="24k"/>
-<part name="R511" library="Passive Components &gt; Resistors &gt; Chip Resistors" deviceset="RESISTOR" device="0603" value="24k"/>
+<part name="R504" library="Passive Components &gt; Resistors &gt; Chip Resistors" deviceset="RESISTOR" device="0603" value="100"/>
+<part name="R505" library="Passive Components &gt; Resistors &gt; Chip Resistors" deviceset="RESISTOR" device="0603" value="10k"/>
+<part name="R510" library="Passive Components &gt; Resistors &gt; Chip Resistors" deviceset="RESISTOR" device="0603" value="10k"/>
+<part name="R511" library="Passive Components &gt; Resistors &gt; Chip Resistors" deviceset="RESISTOR" device="0603" value="10k"/>
 <part name="GND508" library="Utility &gt; Power Symbols" deviceset="GND" device=""/>
 <part name="GND510" library="Utility &gt; Power Symbols" deviceset="GND" device=""/>
